File: KiCad_Files/unicorn.kicad_sch (KiCad schematic)
At the start: 6 parts, among them SW1 SW_DIP_x01

Commit message: pendand 0.1 experiments
Parts:
- removed D4: LED, Binary_Kitchen:5mm_SMD-Pad, symbol Device:LED
- D1, D2, D3: footprint Binary_Kitchen:5mm_SMD-Pad -> LED_THT:LED_D5.0mm_Clear
Changed lines of the file:
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@@
 (kicad_sch
-	(version 20231120)
+	(version 20250114)
 	(generator "eeschema")
-	(generator_version "8.0")
+	(generator_version "9.0")
 	(paper "A4")
-	(junction
-		(at 139.7 82.55)
-		(diameter 0)
-		(color 0 0 0 0)
-	)
-	(junction
-		(at 107.95 82.55)
-		(diameter 0)
-		(color 0 0 0 0)
-	)
 	(junction
 		(at 139.7 72.39)
@@
 	(wire
 		(pts
-			(xy 139.7 93.98) (xy 139.7 82.55)
-		)
-		(stroke
-			(width 0)
-			(type default)
-		)
-	)
-	(wire
-		(pts
 			(xy 107.95 77.47) (xy 104.14 77.47)
 		)
@@
 	(wire
 		(pts
-			(xy 125.73 93.98) (xy 139.7 93.98)
-		)
-		(stroke
-			(width 0)
-			(type default)
-		)
-	)
-	(wire
-		(pts
 			(xy 125.73 82.55) (xy 139.7 82.55)
 		)
@@
 	(wire
 		(pts
-			(xy 107.95 93.98) (xy 107.95 82.55)
-		)
-		(stroke
-			(width 0)
-			(type default)
-		)
-	)
-	(wire
-		(pts
 			(xy 139.7 72.39) (xy 139.7 77.47)
-		)
-		(stroke
-			(width 0)
-			(type default)
-		)
-	)
-	(wire
-		(pts
-			(xy 118.11 93.98) (xy 107.95 93.98)
 		)
 		(stroke
@@
 			)
 		)
-		(property "Footprint" "Binary_Kitchen:5mm_SMD-Pad"
+		(property "Footprint" "LED_THT:LED_D5.0mm_Clear"
 			(at 121.92 62.23 0)
 			(effects
@@
 			)
 		)
-		(property "Footprint" "Binary_Kitchen:5mm_SMD-Pad"
+		(property "Footprint" "LED_THT:LED_D5.0mm_Clear"
 			(at 121.92 72.39 0)
 			(effects
@@
 			)
 		)
-		(property "Footprint" "Binary_Kitchen:5mm_SMD-Pad"
+		(property "Footprint" "LED_THT:LED_D5.0mm_Clear"
 			(at 121.92 82.55 0)
 			(effects
@@
 				(path "/d0939de7-a209-4c8a-aa4c-07879145d509"
 					(reference "D3")
-					(unit 1)
-				)
-			)
-		)
-	)
-	(symbol
-		(lib_id "Device:LED")
-		(at 121.92 93.98 180)
-		(unit 1)
-		(exclude_from_sim no)
-		(in_bom yes)
-		(on_board yes)
-		(dnp no)
-		(property "Reference" "D4"
-			(at 122.0978 99.4918 0)
-			(effects
-				(font
-					(size 1.27 1.27)
-				)
-			)
-		)
-		(property "Value" "LED"
-			(at 122.0978 97.1804 0)
-			(effects
-				(font
-					(size 1.27 1.27)
-				)
-			)
-		)
-		(property "Footprint" "Binary_Kitchen:5mm_SMD-Pad"
-			(at 121.92 93.98 0)
-			(effects
-				(font
-					(size 1.27 1.27)
-				)
-				(hide yes)
-			)
-		)
-		(property "Datasheet" "~"
-			(at 121.92 93.98 0)
-			(effects
-				(font
-					(size 1.27 1.27)
-				)
-				(hide yes)
-			)
-		)
-		(property "Description" ""
-			(at 121.92 93.98 0)
-			(effects
-				(font
-					(size 1.27 1.27)
-				)
-				(hide yes)
-			)
-		)
-		(pin "1"
-		)
-		(pin "2"
-		)
-		(instances
-			(project "unicorn"
-				(path "/d0939de7-a209-4c8a-aa4c-07879145d509"
-					(reference "D4")
 					(unit 1)
 				)
@@
 		)
 	)
+	(embedded_fonts no)
 )
